Commit message: initial commit

File: go2_robot_sdk/urdf/go2.urdf (robot description, URDF)
Before this commit: robot go2, 33 links, 32 joints
Links:
- removed link radar
- added link utlidar_lidar, mass 0
Joints:
- removed joint radar_joint
- added joint utlidar_lidar_joint: type fixed, parent base_link, child utlidar_lidar, origin xyz=0.28945 0 -0.046825 rpy=0 2.8782 0, axis 0 0 0
